Commit message: Updated YOLO perception and Python AI brain scripts

File: MindForgeAI-Project-Master-Workspace/04_active_workspaces/RoboPath_AI_ARGUS/src/robot_description/urdf/argus_robot.urdf (robot description, URDF)
Before this commit: robot argus_robot, 10 links, 9 joints
Links:
- removed link camera_link_optical
Joints:
- removed joint camera_optical_joint
